Commit message: feat: add first base link for arm

File: tf_urdf_rviz_gazebo/my_robot_description/urdf/camera.xacro (robot description, xacro)
@@ -21,4 +21,13 @@
                        o_xyz="0 0 0" o_rpy="0 0 0" />
     </link>
+     <link name="camera_link_optical" />
+     <joint name="camera_optical_joint" type="fixed">
+        <!-- these values have to be these values otherwise the gazebo camera
+            image won't be aligned properly with the frame it is supposedly
+            originating from -->
+        <origin xyz="0 0 0" rpy="${-pi/2} 0 ${-pi/2}"/>
+        <parent link="camera_link"/>
+        <child link="camera_link_optical"/>
+    </joint>
     <joint name="base_camera_joint" type="fixed">
         <parent link="base_link" />
@@ -44,5 +53,5 @@
                     <stddev>0.007</stddev>
                 </noise>
-                <optical_frame_id>camera_link</optical_frame_id>
+                <optical_frame_id>camera_link_optical</optical_frame_id>
                 <camera_info_topic>camera/camera_info</camera_info_topic>
             </camera>

File: tf_urdf_rviz_gazebo/my_robot_description/urdf/common_properties.xacro (robot description, xacro)
@@ -6,4 +6,7 @@
     <material name="grey">
         <color rgba="0.5 0.5 0.5 1" />
+    </material>
+    <material name="green">
+        <color rgba="0.0 1.0 0.0 1" />
     </material>
     <xacro:macro name="box_inertia" params="m x y z o_xyz o_rpy">
