Commit message: feat: add forearm

File: tf_urdf_rviz_gazebo/my_robot_description/urdf/arm.xacro (robot description, xacro)
@@ -4,6 +4,6 @@
     <xacro:property name="arm_base_width" value="0.1" />
     <xacro:property name="arm_base_height" value="0.02" />
-    <!-- <xacro:property name="wheel_radius" value="0.1" /> -->
-    <!-- <xacro:property name="wheel_length" value="0.05" /> -->
+    <xacro:property name="forearm_radius" value="0.02" />
+    <xacro:property name="forearm_length" value="0.3" />
     <link name="arm_base_link">
         <visual>
@@ -20,6 +20,37 @@
             <origin xyz="0 0 0" rpy="0 0 0" />
         </collision>
-        <!-- <xacro:box_inertia m="5.0" x="${base_length}" y="${base_width}" z="${base_height}"
-                       o_xyz="0 0 ${base_height / 2.0}" o_rpy="0 0 0" /> -->
+        <xacro:box_inertia m="5.0" x="${arm_base_length}" y="${arm_base_width}" z="${arm_base_height}"
+                       o_xyz="0 0 0" o_rpy="0 0 0" />
     </link>
+    <link name="forearm_link">
+        <visual>
+            <geometry>
+                <cylinder radius="${forearm_radius}" length="${forearm_length}" />
+            </geometry>
+            <origin xyz="0 0 0" rpy="0 0 0" />
+            <material name="yellow" />
+        </visual>
+        <collision>
+            <geometry>
+                <cylinder radius="${forearm_radius}" length="${forearm_length}" />
+            </geometry>
+            <origin xyz="0 0 0" rpy="0 0 0" />
+        </collision>
+        <xacro:cylinder_inertia m="0.5" r="${forearm_radius}" l="${forearm_length}"
+                    o_xyz="0 0 0" o_rpy="0 0 0" />
+    </link>
+    <joint name="arm_base_joint" type="fixed">
+        <parent link="base_footprint" />
+        <child link="arm_base_link" />
+        <origin xyz="1.0 0 0" rpy="0 0 0"/>
+    </joint>
+    <joint name="arm_base_forearm_joint" type="revolute">
+        <parent link="arm_base_link" />
+        <child link="forearm_link" />
+        <origin xyz="0 0 ${(arm_base_height / 2.0) + (forearm_length / 2.0)}" rpy="0 0 0"/>
+        <!-- <origin xyz="0 0 3" rpy="0 0 0"/> -->
+        <axis xyz="0 0 1" />
+        <limit lower="0" upper="${pi / 2.0}" effort="100" velocity="100" />
+        <dynamics damping="0.3" friction="0.3" />
+    </joint>
 </robot>

File: tf_urdf_rviz_gazebo/my_robot_description/urdf/common_properties.xacro (robot description, xacro)
@@ -9,4 +9,7 @@
     <material name="green">
         <color rgba="0.0 1.0 0.0 1" />
+    </material>
+     <material name="yellow">
+        <color rgba="1.0 1.0 0.0 1" />
     </material>
     <xacro:macro name="box_inertia" params="m x y z o_xyz o_rpy">

Commit message: feat: add hand

File: tf_urdf_rviz_gazebo/my_robot_description/urdf/arm.xacro (robot description, xacro)
@@ -4,5 +4,5 @@
     <xacro:property name="arm_base_width" value="0.1" />
     <xacro:property name="arm_base_height" value="0.02" />
-    <xacro:property name="forearm_radius" value="0.02" />
+    <xacro:property name="forearm_hand_radius" value="0.02" />
     <xacro:property name="forearm_length" value="0.3" />
     <link name="arm_base_link">
@@ -26,5 +26,5 @@
         <visual>
             <geometry>
-                <cylinder radius="${forearm_radius}" length="${forearm_length}" />
+                <cylinder radius="${forearm_hand_radius}" length="${forearm_length}" />
             </geometry>
             <origin xyz="0 0 0" rpy="0 0 0" />
@@ -33,9 +33,26 @@
         <collision>
             <geometry>
-                <cylinder radius="${forearm_radius}" length="${forearm_length}" />
+                <cylinder radius="${forearm_hand_radius}" length="${forearm_length}" />
             </geometry>
             <origin xyz="0 0 0" rpy="0 0 0" />
         </collision>
-        <xacro:cylinder_inertia m="0.5" r="${forearm_radius}" l="${forearm_length}"
+        <xacro:cylinder_inertia m="0.5" r="${forearm_hand_radius}" l="${forearm_length}"
+                    o_xyz="0 0 0" o_rpy="0 0 0" />
+    </link>
+     <link name="hand_link">
+        <visual>
+            <geometry>
+                <cylinder radius="${forearm_hand_radius}" length="${forearm_length}" />
+            </geometry>
+            <origin xyz="0 0 0" rpy="0 0 0" />
+            <material name="yellow" />
+        </visual>
+        <collision>
+            <geometry>
+                <cylinder radius="${forearm_hand_radius}" length="${forearm_length}" />
+            </geometry>
+            <origin xyz="0 0 0" rpy="0 0 0" />
+        </collision>
+        <xacro:cylinder_inertia m="0.5" r="${forearm_hand_radius}" l="${forearm_length}"
                     o_xyz="0 0 0" o_rpy="0 0 0" />
     </link>
@@ -49,6 +66,13 @@
         <child link="forearm_link" />
         <origin xyz="0 0 ${(arm_base_height / 2.0) + (forearm_length / 2.0)}" rpy="0 0 0"/>
-        <!-- <origin xyz="0 0 3" rpy="0 0 0"/> -->
-        <axis xyz="0 0 1" />
+        <axis xyz="0 1 0" />
+        <limit lower="0" upper="${pi / 2.0}" effort="100" velocity="100" />
+        <dynamics damping="0.3" friction="0.3" />
+    </joint>
+     <joint name="hand_forearm_joint" type="revolute">
+        <parent link="forearm_link" />
+        <child link="hand_link" />
+        <origin xyz="0 0 ${(arm_base_height / 2.0) + forearm_length}" rpy="0 0 0"/>
+        <axis xyz="0 1 0" />
         <limit lower="0" upper="${pi / 2.0}" effort="100" velocity="100" />
         <dynamics damping="0.3" friction="0.3" />

Commit message: feat: adapt position for right moving

File: tf_urdf_rviz_gazebo/my_robot_description/urdf/arm.xacro (robot description, xacro)
@@ -28,5 +28,5 @@
                 <cylinder radius="${forearm_hand_radius}" length="${forearm_length}" />
             </geometry>
-            <origin xyz="0 0 0" rpy="0 0 0" />
+            <origin xyz="${(forearm_hand_radius / 2.0)} ${(forearm_hand_radius / 2.0)} ${(forearm_length / 2.0)}" rpy="0 0 0" />
             <material name="yellow" />
         </visual>
@@ -35,5 +35,5 @@
                 <cylinder radius="${forearm_hand_radius}" length="${forearm_length}" />
             </geometry>
-            <origin xyz="0 0 0" rpy="0 0 0" />
+            <origin xyz="${(forearm_hand_radius / 2.0)} ${(forearm_hand_radius / 2.0)} ${(forearm_length / 2.0)}" rpy="0 0 0" />
         </collision>
         <xacro:cylinder_inertia m="0.5" r="${forearm_hand_radius}" l="${forearm_length}"
@@ -45,5 +45,5 @@
                 <cylinder radius="${forearm_hand_radius}" length="${forearm_length}" />
             </geometry>
-            <origin xyz="0 0 0" rpy="0 0 0" />
+            <origin xyz="${(forearm_hand_radius / 2.0)} ${(forearm_hand_radius / 2.0)} ${(forearm_length / 2.0)}" rpy="0 0 0" />
             <material name="yellow" />
         </visual>
@@ -65,5 +65,6 @@
         <parent link="arm_base_link" />
         <child link="forearm_link" />
-        <origin xyz="0 0 ${(arm_base_height / 2.0) + (forearm_length / 2.0)}" rpy="0 0 0"/>
+        <!-- <origin xyz="0 0 ${(arm_base_height / 2.0) + (forearm_length / 2.0)}" rpy="0 0 0"/> -->
+        <origin xyz="0 0 0" rpy="0 0 0"/>
         <axis xyz="0 1 0" />
         <limit lower="0" upper="${pi / 2.0}" effort="100" velocity="100" />
@@ -73,5 +74,6 @@
         <parent link="forearm_link" />
         <child link="hand_link" />
-        <origin xyz="0 0 ${(arm_base_height / 2.0) + forearm_length}" rpy="0 0 0"/>
+        <!-- <origin xyz="0 0 ${(arm_base_height / 2.0) + forearm_length}" rpy="0 0 0"/> -->
+        <origin xyz="0 0 ${forearm_length}" rpy="0 0 0"/>
         <axis xyz="0 1 0" />
         <limit lower="0" upper="${pi / 2.0}" effort="100" velocity="100" />

Commit message: feat: finish project

File: tf_urdf_rviz_gazebo/my_robot_description/urdf/arm.xacro (robot description, xacro)
@@ -58,13 +58,12 @@
     </link>
     <joint name="arm_base_joint" type="fixed">
-        <parent link="base_footprint" />
+        <parent link="base_link" />
         <child link="arm_base_link" />
-        <origin xyz="1.0 0 0" rpy="0 0 0"/>
+        <origin xyz="0 0 ${base_height + (arm_base_height / 2.0)}" rpy="0 0 0"/>
     </joint>
     <joint name="arm_base_forearm_joint" type="revolute">
         <parent link="arm_base_link" />
         <child link="forearm_link" />
-        <!-- <origin xyz="0 0 ${(arm_base_height / 2.0) + (forearm_length / 2.0)}" rpy="0 0 0"/> -->
-        <origin xyz="0 0 0" rpy="0 0 0"/>
+        <origin xyz="0 0 ${(arm_base_height / 2.0)}" rpy="0 0 0"/>
         <axis xyz="0 1 0" />
         <limit lower="0" upper="${pi / 2.0}" effort="100" velocity="100" />
@@ -74,5 +73,4 @@
         <parent link="forearm_link" />
         <child link="hand_link" />
-        <!-- <origin xyz="0 0 ${(arm_base_height / 2.0) + forearm_length}" rpy="0 0 0"/> -->
         <origin xyz="0 0 ${forearm_length}" rpy="0 0 0"/>
         <axis xyz="0 1 0" />
